Commit message: Added myball to myworld. Added materials.xacro and colors to my_robot.xacro.

File: my_robot/urdf/my_robot.xacro (robot description, xacro)
@@ -2,4 +2,5 @@
 <robot name="my_robot" xmlns:xacro="http://www.ros.org/wiki/xacro">
   <xacro:include filename="$(find my_robot)/urdf/my_robot.gazebo" />
+  <xacro:include filename="$(find my_robot)/urdf/materials.xacro" />
   <link name="robot_footprint"></link>
   <joint name="robot_footprint_joint" type="fixed">
@@ -30,4 +31,5 @@
         <box size=".4 .2 .1"/>
       </geometry>
+      <material name="orange"/>
     </visual>
     <collision name='back_caster_collision'>
@@ -42,4 +44,5 @@
         <sphere radius="0.05"/>
       </geometry>
+      <material name="silver"/>
     </visual>
     <collision name='front_caster_collision'>

Commit message: Fixed misspelling.

File: my_robot/urdf/my_robot.xacro (robot description, xacro)
@@ -65,5 +65,5 @@
       <origin xyz="0 0 0" rpy="0 0 0"/>
       <inertia ixx="1e-6" ixy="0" ixz="0" iyy="1e-6" iyz="0" izz="1e-6"/>
-    </inertia>
+    </inertial>
     <collision name='collision'>
       <origin xyz="0 0 0"/>

Commit message: Add wheels and correct colors to the robot.

File: my_robot/urdf/my_robot.xacro (robot description, xacro)
@@ -31,5 +31,7 @@
         <box size=".4 .2 .1"/>
       </geometry>
-      <material name="orange"/>
+      <material name="orange">
+        <color rgba="${255/255} ${165/255} ${0/255} 1.0"/>
+      </material>
     </visual>
     <collision name='back_caster_collision'>
@@ -44,5 +46,7 @@
         <sphere radius="0.05"/>
       </geometry>
-      <material name="silver"/>
+      <material name="silver">
+        <color rgba="${192/255} ${192/255} ${192/255} 1.0"/>
+      </material>
     </visual>
     <collision name='front_caster_collision'>
@@ -57,4 +61,7 @@
         <sphere radius="0.05"/>
       </geometry>
+      <material name="silver">
+        <color rgba="${192/255} ${192/255} ${192/255} 1.0"/>
+      </material>
     </visual>
   </link>
@@ -87,4 +94,5 @@
     <dynamics damping="1.0" friction="1.0"/>
   </joint>
+  <!-- hokuyo lidar -->
   <link name='hokuyo'>
     <pose>0 0 0 0 0</pose>
@@ -115,3 +123,69 @@
     <dynamics damping="1.0" friction="1.0"/>
   </joint>
+  <!-- LEFT WHEEL LINK -->
+  <link name="left_wheel">
+    <pose>0 0 0 0 0</pose>
+    <inertial>
+      <mass value="5"/>
+      <origin xyz="0 0 0" rpy="0 1.5707 1.5707"/>
+      <inertia  ixx="0.1" ixy="0" ixz="0"
+                iyy="0.1" iyz="0" izz="0.1"/>
+    </inertial>
+    <collision name='collision'>
+      <origin xyz="0.0 0 0.0" rpy="0 1.5707 1.5707"/>
+      <geometry>
+        <cylinder radius="0.1" length="0.05"/>
+      </geometry>
+    </collision>
+    <visual name='visual'>
+      <origin xyz="0 0 0" rpy="0 1.5707 1.5707"/>
+      <geometry>
+        <cylinder radius="0.1" length="0.05"/>
+      </geometry>
+    </visual>
+    <material name="brown">
+      <color rgba="${139/255} ${69/255} ${19/255} 1.0"/>
+    </material>
+  </link>
+  <joint type="continuous" name="left_wheel_hinge">
+    <origin xyz="0 0.15 0" rpy="0 0 0"/>
+    <child link="left_wheel"/>
+    <parent link="chassis"/>
+    <axis xyz="0 1 0" rpy="0 0 0"/>
+    <limit effort="10000" velocity="1000"/>
+    <dynamics damping="1.0" friction="1.0"/>
+  </joint>
+  <!-- RIGHT WHEEN LINK -->
+  <link name="right_wheel">
+    <pose>0 0 0 0 0</pose>
+    <inertial>
+      <mass value="5"/>
+      <origin xyz="0 0 0" rpy="0 1.5707 1.5707"/>
+      <inertia  ixx="0.1" ixy="0" ixz="0"
+                iyy="0.1" iyz="0" izz="0.1"/>
+    </inertial>
+    <collision name='collision'>
+      <origin xyz="0 0 0" rpy="0 1.5707 1.5707"/>
+      <geometry>
+        <cylinder radius="0.1" length="0.05"/>
+      </geometry>
+    </collision>
+    <visual name='visual'>
+      <origin xyz="0 0 0" rpy="0 0 0"/>
+      <geometry>
+        <cylinder radius="0.1" length="0.05"/>
+      </geometry>
+    </visual>
+    <material name="brown">
+      <color rgba="${139/255} ${69/255} ${19/255} 1.0"/>
+    </material>
+  </link>
+  <joint type="continuous" name="right_wheel_hinge">
+    <origin xyz="0 -0.15 0" rpy="0 0 0"/>
+    <child link="right_wheel"/>
+    <parent link="chassis"/>
+    <axis xyz="0 1 0" rpy="0 0 0"/>
+    <limit effort="10000" velocity="1000"/>
+    <dynamics damping="1.0" friction="1.0"/>
+  </joint>
 </robot>

Commit message: Fix right wheel so that it looks vertical.

File: my_robot/urdf/my_robot.xacro (robot description, xacro)
@@ -172,5 +172,5 @@
     </collision>
     <visual name='visual'>
-      <origin xyz="0 0 0" rpy="0 0 0"/>
+      <origin xyz="0 0 0" rpy="0 1.5707 1.5707"/>
       <geometry>
         <cylinder radius="0.1" length="0.05"/>

Commit message: Add colors to the model.

File: my_robot/urdf/my_robot.xacro (robot description, xacro)
@@ -189,3 +189,13 @@
     <dynamics damping="1.0" friction="1.0"/>
   </joint>
+  <!-- colors for chasis and wheels -->
+  <gazebo reference="chassis">
+    <material>Gazebo/Orange</material>
+  </gazebo>
+  <gazebo reference="left_wheel">
+    <material>Gazebo/Green</material>
+  </gazebo>
+  <gazebo reference="right_wheel">
+    <material>Gazebo/Red</material>
+  </gazebo>
 </robot>

Commit message: Eliminate a name attribute conflict.

File: my_robot/urdf/my_robot.xacro (robot description, xacro)
@@ -46,7 +46,4 @@
         <sphere radius="0.05"/>
       </geometry>
-      <material name="silver">
-        <color rgba="${192/255} ${192/255} ${192/255} 1.0"/>
-      </material>
     </visual>
     <collision name='front_caster_collision'>
@@ -61,7 +58,4 @@
         <sphere radius="0.05"/>
       </geometry>
-      <material name="silver">
-        <color rgba="${192/255} ${192/255} ${192/255} 1.0"/>
-      </material>
     </visual>
   </link>
@@ -125,5 +119,4 @@
   <!-- LEFT WHEEL LINK -->
   <link name="left_wheel">
-    <pose>0 0 0 0 0</pose>
     <inertial>
       <mass value="5"/>
@@ -132,5 +125,5 @@
                 iyy="0.1" iyz="0" izz="0.1"/>
     </inertial>
-    <collision name='collision'>
+    <collision>
       <origin xyz="0.0 0 0.0" rpy="0 1.5707 1.5707"/>
       <geometry>
@@ -138,5 +131,5 @@
       </geometry>
     </collision>
-    <visual name='visual'>
+    <visual>
       <origin xyz="0 0 0" rpy="0 1.5707 1.5707"/>
       <geometry>
@@ -144,7 +137,4 @@
       </geometry>
     </visual>
-    <material name="brown">
-      <color rgba="${139/255} ${69/255} ${19/255} 1.0"/>
-    </material>
   </link>
   <joint type="continuous" name="left_wheel_hinge">
@@ -158,5 +148,4 @@
   <!-- RIGHT WHEEN LINK -->
   <link name="right_wheel">
-    <pose>0 0 0 0 0</pose>
     <inertial>
       <mass value="5"/>
@@ -165,5 +154,5 @@
                 iyy="0.1" iyz="0" izz="0.1"/>
     </inertial>
-    <collision name='collision'>
+    <collision>
       <origin xyz="0 0 0" rpy="0 1.5707 1.5707"/>
       <geometry>
@@ -171,5 +160,5 @@
       </geometry>
     </collision>
-    <visual name='visual'>
+    <visual>
       <origin xyz="0 0 0" rpy="0 1.5707 1.5707"/>
       <geometry>
@@ -177,7 +166,4 @@
       </geometry>
     </visual>
-    <material name="brown">
-      <color rgba="${139/255} ${69/255} ${19/255} 1.0"/>
-    </material>
   </link>
   <joint type="continuous" name="right_wheel_hinge">

Commit message: Change my robot shape. Fix process image loop and right cutoff value.

File: my_robot/urdf/my_robot.xacro (robot description, xacro)
@@ -20,5 +20,5 @@
       />
     </inertial>
-    <collision name='collision'>
+    <collision name='collision_vertical'>
       <origin xyz="0 0 0" rpy=" 0 0 0"/>
       <geometry>
@@ -26,5 +26,5 @@
       </geometry>
     </collision>
-    <visual name='chassis_visual'>
+    <visual name='chassis_visual_vertical'>
       <origin xyz="0 0 0" rpy=" 0 0 0"/>
       <geometry>
@@ -35,8 +35,23 @@
       </material>
     </visual>
+    <collision name='collision_horizontal'>
+      <origin xyz="0 0 0" rpy=" 0 0 0"/>
+      <geometry>
+        <box size=".1 .4 .1"/>
+      </geometry>
+    </collision>
+    <visual name='chassis_visual_horizontal'>
+      <origin xyz="0 0 0" rpy=" 0 0 0"/>
+      <geometry>
+        <box size=".1 .4 .1"/>
+      </geometry>
+      <material name="orange">
+        <color rgba="${255/255} ${165/255} ${0/255} 1.0"/>
+      </material>
+    </visual>
     <collision name='back_caster_collision'>
       <origin xyz="-0.15 0 -0.05" rpy=" 0 0 0"/>
       <geometry>
-        <sphere radius="0.0499"/>
+        <sphere radius="0.05"/>
       </geometry>
     </collision>
@@ -50,5 +65,5 @@
       <origin xyz="0.15 0 -0.05" rpy=" 0 0 0"/>
       <geometry>
-        <sphere radius="0.0499"/>
+        <sphere radius="0.05"/>
       </geometry>
     </collision>
@@ -139,5 +154,5 @@
   </link>
   <joint type="continuous" name="left_wheel_hinge">
-    <origin xyz="0 0.15 0" rpy="0 0 0"/>
+    <origin xyz="0 0.225 0" rpy="0 0 0"/>
     <child link="left_wheel"/>
     <parent link="chassis"/>
@@ -168,5 +183,5 @@
   </link>
   <joint type="continuous" name="right_wheel_hinge">
-    <origin xyz="0 -0.15 0" rpy="0 0 0"/>
+    <origin xyz="0 -0.225 0" rpy="0 0 0"/>
     <child link="right_wheel"/>
     <parent link="chassis"/>

Commit message: Fixing origin of hokuyo collision to be the same as the inertial and visual.

File: my_robot/urdf/my_robot.xacro (robot description, xacro)
@@ -112,5 +112,5 @@
     </inertial>
     <collision name='collision'>
-      <origin xyz="0.15 0 0.1" rpy="0 0 0"/>
+      <origin xyz="0 0 0" rpy="0 0 0"/>
       <geometry>
         <box size="0.2 0.2 0.2"/>

Commit message: modifying position and size of hokuyo so it won't scan its own box and it is high enough

File: my_robot/urdf/my_robot.xacro (robot description, xacro)
@@ -112,11 +112,11 @@
     </inertial>
     <collision name='collision'>
-      <origin xyz="0 0 0" rpy="0 0 0"/>
-      <geometry>
-        <box size="0.2 0.2 0.2"/>
+      <origin xyz="0.08 0 0.08" rpy="0 0 0"/>
+      <geometry>
+        <box size="0.05 0.05 0.05"/>
       </geometry>
     </collision>
     <visual name='visual'>
-      <origin xyz="0 0 0" rpy="0 0 0"/>
+      <origin xyz="0.08 0 0.08" rpy="0 0 0"/>
       <geometry>
         <mesh filename="package://my_robot/mesh_files/hokuyo.dae"/>
@@ -125,5 +125,5 @@
   </link>
   <joint type="fixed" name="hokuyo_joint">
-    <origin xyz="0.15 0 0.1" rpy="0 0 0"/>
+    <origin xyz="0.08 0 0.08" rpy="0 0 0"/>
     <child link="hokuyo"/>
     <parent link="chassis"/>

Commit message: Initial commits for the map-my-world project.

File: my_robot/urdf/my_robot.xacro (robot description, xacro)
@@ -75,5 +75,5 @@
     </visual>
   </link>
-  <link name='camera'>
+  <link name='camera_link'>
     <pose>0 0 0 0 0</pose>
     <inertial>
@@ -82,5 +82,5 @@
       <inertia ixx="1e-6" ixy="0" ixz="0" iyy="1e-6" iyz="0" izz="1e-6"/>
     </inertial>
-    <collision name='collision'>
+    <collision name='camera_link_collision'>
       <origin xyz="0 0 0"/>
       <geometry>
@@ -88,5 +88,5 @@
       </geometry>
     </collision>
-    <visual name='visual'>
+    <visual name='camera_link_visual'>
       <origin xyz="0 0 0"/>
       <geometry>
@@ -97,5 +97,5 @@
   <joint type="fixed" name="camera_joint">
     <origin xyz="0.2 0 0" rpy="0 0 0"/>
-    <child link="camera"/>
+    <child link="camera_link"/>
     <parent link="chassis"/>
     <axis xyz="0 1 0" rpy="0 0 0"/>
@@ -103,4 +103,12 @@
     <dynamics damping="1.0" friction="1.0"/>
   </joint>
+  <!-- optical camera link (project 4 map my world) -->
+  <joint name="camera_optical_joint" type="fixed">
+    <origin xyz="0 0 0" rpy="-1.5707 0 -1.5707"/>
+    <parent link="camera_link"/>
+    <child link="camera_link_optical"/>
+  </joint>
+  <link name="camera_link_optical">
+  </link>
   <!-- hokuyo lidar -->
   <link name='hokuyo'>

Commit message: Decreasing the sphere radius of the front and back casters so that the wheels can move the robot and the casters don't create too much friction for the robot.

File: my_robot/urdf/my_robot.xacro (robot description, xacro)
@@ -53,5 +53,5 @@
       <origin xyz="-0.15 0 -0.05" rpy=" 0 0 0"/>
       <geometry>
-        <sphere radius="0.05"/>
+        <sphere radius="0.0495"/>
       </geometry>
     </collision>
@@ -59,5 +59,5 @@
       <origin xyz="-0.15 0 -0.05" rpy=" 0 0 0"/>
       <geometry>
-        <sphere radius="0.05"/>
+        <sphere radius="0.0495"/>
       </geometry>
     </visual>
@@ -65,5 +65,5 @@
       <origin xyz="0.15 0 -0.05" rpy=" 0 0 0"/>
       <geometry>
-        <sphere radius="0.05"/>
+        <sphere radius="0.0495"/>
       </geometry>
     </collision>
@@ -71,5 +71,5 @@
       <origin xyz="0.15 0 -0.05" rpy=" 0 0 0"/>
       <geometry>
-        <sphere radius="0.05"/>
+        <sphere radius="0.0495"/>
       </geometry>
     </visual>

Commit message: Decreasing the size of the casters underneath the robot for less friction to get faster movement.

File: my_robot/urdf/my_robot.xacro (robot description, xacro)
@@ -53,5 +53,5 @@
       <origin xyz="-0.15 0 -0.05" rpy=" 0 0 0"/>
       <geometry>
-        <sphere radius="0.0495"/>
+        <sphere radius="0.049"/>
       </geometry>
     </collision>
@@ -59,5 +59,5 @@
       <origin xyz="-0.15 0 -0.05" rpy=" 0 0 0"/>
       <geometry>
-        <sphere radius="0.0495"/>
+        <sphere radius="0.049"/>
       </geometry>
     </visual>
@@ -65,5 +65,5 @@
       <origin xyz="0.15 0 -0.05" rpy=" 0 0 0"/>
       <geometry>
-        <sphere radius="0.0495"/>
+        <sphere radius="0.049"/>
       </geometry>
     </collision>
@@ -71,5 +71,5 @@
       <origin xyz="0.15 0 -0.05" rpy=" 0 0 0"/>
       <geometry>
-        <sphere radius="0.0495"/>
+        <sphere radius="0.049"/>
       </geometry>
     </visual>
